File: rp2040_bt_feather.kicad_sch (KiCad schematic)
At the start: 70 parts, among them J1 HRO TYPE-C-31-M-12, J2 LIPO_JSTPH, J3 Conn_01x16, J4 Conn_01x12, J5 Qwiic/STEMMA QT, J6 SWD, Q1 DMG3415U-7?, Q2 DMG3415U-7?, SW1 SW_Push, SW2 SW_Push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

Commit message: Lay out power input and supporting passives
Parts:
- removed J5: Qwiic/STEMMA QT, Connector_JST:JST_SH_SM04B-SRSS-TB_1x04-1MP_P1.00mm_Horizontal, symbol Connector_Generic_MountingPin:Conn_01x04_MountingPin
- added FID1, FID2: Fiducial, Fiducial:Fiducial_1mm_Mask2mm, symbol Mechanical:Fiducial
- added H1, H2, H3, H4: MountingHole, MountingHole:MountingHole_2.5mm, symbol Mechanical:MountingHole
- Q1, Q2: symbol Device:Q_PMOS_DGS -> Device:Q_PMOS_GSD
Connections:
- net +3V3: now also Q2.2 (S); no longer Q2.3 (S)
- net +BATT: now also J2.1 (Pin_1), Q1.3 (D); no longer J2.2 (Pin_2), Q1.1 (D)
- net DA_PWR: now also Q2.1 (G); no longer Q2.2 (G)
- net DA_VIN: now also Q2.3 (D); no longer Q2.1 (D)
- net GND: now also J2.2 (Pin_2); no longer J2.1 (Pin_1)
- net VUSB: now also Q1.1 (G); no longer Q1.2 (G)
- net V_IN: now also Q1.2 (S); no longer Q1.3 (S)
Other:
- note added: "TODO: Include filter?"
- note removed: "Qwiic/ Stemma QT"
